Commit message: refactor: rover urdf file links and joints refactored

File: urdf/src/robot/urdf/mark_two.urdf (robot description, URDF)
Before this commit: robot rover, 5 links, 4 joints
Links:
- added link robot_footprint
Joints:
- added joint base_joint: type fixed, parent robot_footprint, child base_link, origin xyz=0.0 0.0 0.1 rpy=0.0 0.0 0.0
- joint base_left_back_wheel: child left_back_wheel -> right_back_wheel; origin xyz=-0.2 -0.225 0.1 rpy=0.0 0.0 0.0 -> xyz=-0.2 0.225 0.0 rpy=0.0 0.0 0.0
- joint base_left_front_wheel: child left_front_wheel -> right_front_wheel; origin xyz=0.2 -0.225 0.1 rpy=0.0 0.0 0.0 -> xyz=0.2 0.225 0.0 rpy=0.0 0.0 0.0
- joint base_right_back_wheel: child right_back_wheel -> left_back_wheel; origin xyz=-0.2 0.225 0.1 rpy=0.0 0.0 0.0 -> xyz=-0.2 -0.225 0.0 rpy=0.0 0.0 0.0
- joint base_right_front_wheel: child right_front_wheel -> left_front_wheel; origin xyz=0.2 0.225 0.1 rpy=0.0 0.0 0.0 -> xyz=0.2 -0.225 0.0 rpy=0.0 0.0 0.0

Commit message: chore: collision property added

File: urdf/src/robot/urdf/mark_two.urdf (robot description, URDF)
Before this commit: robot rover, 6 links, 5 joints
Links:
- link base_link: mass None -> 5.0; geometry collision box size=0.8 0.4 0.1; visual box size=0.8 0.4 0.1
- link left_back_wheel: geometry collision cylinder length=0.05 radius=0.1; visual cylinder length=0.05 radius=0.1
- link left_front_wheel: geometry collision cylinder length=0.05 radius=0.1; visual cylinder length=0.05 radius=0.1
- link right_back_wheel: geometry collision cylinder length=0.05 radius=0.1; visual cylinder length=0.05 radius=0.1
- link right_front_wheel: geometry collision cylinder length=0.05 radius=0.1; visual cylinder length=0.05 radius=0.1
