Commit message: refactor: xacro file code refactored, clubed wheel macro with link and joint together, remove base_link_share macro

File: urdf/src/robot/urdf/mark_three.urdf.xacro (robot description, xacro)
@@ -17,13 +17,6 @@
     <xacro:material name="black" color="0.0 0.0 0.0 1.0" />
     <xacro:material name="white" color="1.0 1.0 1.0 1.0" />
-    <!-- default-inertial -->
-    <xacro:macro name="default_inertial" params="mass">
-        <inertial>
-            <mass value="${mass}" />
-            <inertia ixx="0.0" ixy="0.0" ixz="0.0" iyy="0.0" iyz="0.0" izz="0.0" />
-        </inertial>
-    </xacro:macro>
-    <!-- robot-wheel -->
-    <xacro:macro name="robot_wheel" params="wheel_position">
+    <!-- wheel-macro -->
+    <xacro:macro name="wheel" params="wheel_position reflect_x reflect_y parent">
         <link name="${wheel_position}_wheel">
             <visual>
@@ -41,7 +34,4 @@
             </collision>
         </link>
-    </xacro:macro>
-    <!-- wheel-joints -->
-    <xacro:macro name="wheel_joint" params="wheel_position reflect_x reflect_y parent">
         <joint name="base_${wheel_position}_wheel" type="continuous">
             <origin
@@ -56,26 +46,22 @@
     <link name="robot_footprint" />
     <!-- base-link -->
-    <xacro:macro name="base_link_shape">
-        <geometry>
-            <box size="${length} ${breadth} ${height}" />
-            <origin xyz="0.0 0.0 0.0" />
-        </geometry>
-    </xacro:macro>
     <link name="base_link">
         <visual>
-            <xacro:base_link_shape />
+            <geometry>
+                <box size="${length} ${breadth} ${height}" />
+            </geometry>
             <material name="white" />
         </visual>
         <collision>
-            <xacro:base_link_shape />
+            <geometry>
+                <box size="${length} ${breadth} ${height}" />
+            </geometry>
         </collision>
-        <xacro:default_inertial mass="${base_mass}" />
+        <inertial>
+            <mass value="${base_mass}" />
+            <inertia ixx="0.0" ixy="0.0" ixz="0.0" iyy="0.0" iyz="0.0" izz="0.0" />
+        </inertial>
     </link>
-    <!-- links -->
-    <xacro:robot_wheel wheel_position="left_front" />
-    <xacro:robot_wheel wheel_position="right_front" />
-    <xacro:robot_wheel wheel_position="left_back" />
-    <xacro:robot_wheel wheel_position="right_back" />
-    <!-- joints -->
+    <!-- base-joint -->
     <joint name="base_joint" type="fixed">
         <parent link="robot_footprint" />
@@ -83,7 +69,8 @@
         <origin xyz="0.0 0.0 0.1" rpy="0.0 0.0 0.0" />
     </joint>
-    <xacro:wheel_joint wheel_position="left_front" reflect_x="1.0" reflect_y="1.0" parent="base_link" />
-    <xacro:wheel_joint wheel_position="right_front" reflect_x="1.0" reflect_y="-1.0" parent="base_link" />
-    <xacro:wheel_joint wheel_position="left_back" reflect_x="-1.0" reflect_y="1.0" parent="base_link" />
-    <xacro:wheel_joint wheel_position="right_back" reflect_x="-1.0" reflect_y="-1.0" parent="base_link" />
+    <!-- wheels -->
+    <xacro:wheel wheel_position="left_front" reflect_x="1.0" reflect_y="1.0" parent="base_link" />
+    <xacro:wheel wheel_position="right_front" reflect_x="1.0" reflect_y="-1.0" parent="base_link" />
+    <xacro:wheel wheel_position="left_back" reflect_x="-1.0" reflect_y="1.0" parent="base_link" />
+    <xacro:wheel wheel_position="right_back" reflect_x="-1.0" reflect_y="-1.0" parent="base_link" />
 </robot>
